File: kicad/scbs_demo/scbs_demo.kicad_sch (KiCad schematic)
At the start: 33 parts

Commit message: scbs_pico hardware Rev A, initial firmware
Parts:
- removed C?: DNP, symbol Device:C
- removed C?: 10uF, symbol Device:C
- removed J?: Conn_01x02_Male, symbol Connector:Conn_01x02_Male
- removed Q?: 2N3904, Package_TO_SOT_THT:TO-92_Inline, symbol Transistor_BJT:2N3904
- removed R?: 10k, symbol Device:R_US
- removed U? (x3): LM358, symbol Amplifier_Operational:LM358
- added C1, C7, C8: 0.1uF, Capacitor_SMD:C_0805_2012Metric, symbol Device:C
- added D1, D2, D3: 1N4148, Diode_SMD:D_SOD-123, symbol Device:D
- added GRAPHIC1: Graphic, Custom_Graphic:bird_with_pants_small_flipped, symbol Custom_Placeholder:Graphic
- added H1: MountingHole, MountingHole:MountingHole_3.2mm_M3, symbol Mechanical:MountingHole
- added J1: Conn_01x06_Male, Connector_PinHeader_2.54mm:PinHeader_1x06_P2.54mm_Horizontal, symbol Connector:Conn_01x06_Male
- added J2: Conn_ARM_JTAG_SWD_10, Connector_PinHeader_1.27mm:PinHeader_2x05_P1.27mm_Vertical_SMD, symbol Connector:Conn_ARM_JTAG_SWD_10
- added PCB1: PCB, Custom_Graphic:PCB_PN_REV_small, symbol Custom_Placeholder:PCB
- added Q2: 2N7002, Package_TO_SOT_SMD:SOT-23, symbol Transistor_FET:2N7002
- added Q4: MMBT3904, Package_TO_SOT_SMD:SOT-23, symbol Transistor_BJT:MMBT3904
- added R1, R20: 2k, Resistor_SMD:R_0805_2012Metric, symbol Device:R_US
- added R11, R15, R25, R30: 10k, Resistor_SMD:R_0805_2012Metric, symbol Device:R_US
- added R19: 1R, Resistor_SMD:R_0805_2012Metric, symbol Device:R_US
- added R23, R24, R6: 390R, Resistor_SMD:R_0805_2012Metric, symbol Device:R_US
- added R3, R4: 3k3, Resistor_SMD:R_0805_2012Metric, symbol Device:R_US
- added TP1, TP10, TP11, TP2, TP3, TP4, TP5, TP6, TP7, TP8, TP9: TestPoint, TestPoint:TestPoint_Pad_2.0x2.0mm, symbol Connector:TestPoint
- added U1: TLV9062xD, Package_SO:SOIC-8_3.9x4.9mm_P1.27mm, symbol Amplifier_Operational:TLV9062xD
- added U2: PC817, Package_DIP:DIP-4_W7.62mm, symbol Isolator:PC817
- added U3: Pico, Custom_Module:RPi_Pico_SMD_TH, symbol Custom_MCU:Pico
- C2, C3, C4, C5, C6: renamed from C?; footprint (none) -> Capacitor_SMD:C_0805_2012Metric; Standard Cost (none) -> 0.10
- C9: renamed from C?; value 10uF -> 0.1uF; footprint (none) -> Capacitor_SMD:C_0805_2012Metric; Standard Cost (none) -> 0.10
- Q1: renamed from Q?; footprint (none) -> Package_TO_SOT_THT:TO-92; MPN (none) -> PN2907ATF; Standard Cost (none) -> 0.07
- Q3: renamed from Q?; Standard Cost (none) -> 0.04
- R10, R12, R13, R14, R16, R17, R18, R2, R21, R22, R26, R27, R28, R7, R8, R9: renamed from R?; footprint (none) -> Resistor_SMD:R_0805_2012Metric; Standard Cost (none) -> 0.01
- R5: renamed from R?; value 0R -> 100R; footprint (none) -> Resistor_SMD:R_0805_2012Metric; Standard Cost (none) -> 0.01
Connections:
- net +5V: now also D1.1 (K), J1.1 (Pin_1), R3.1, TP10.1, U1.8 (V+), U3.39 (VSYS)
- net CMD: now also R15.1, TP2.1
- net CMD_PWM: now also TP4.1, U3.21 (GPIO16)
- net CSENSE: now also R25.1, TP8.1, U1.7
- net GND: now also C7.2, C8.2, D2.2 (A), J1.3 (Pin_3), J2.3 (GND), J2.5 (GND), Q4.2 (E), R19.2, R20.2, R24.2, TP9.1, U1.4 (V-), U3.28 (GND), U3.3 (GND), U3.33 (AGND), U3.38 (GND), U3.42 (GND); no longer Q3.2 (E)
- net OUT: now also J1.2 (Pin_2), TP6.1
- net SHUNT_HI: now reaches C5.1, Q1.1 (C), R10.1, R12.1, R14.1, R17.1, R8.1, R9.1
- net SHUNT_HI: now also TP1.1
- net BASE: now reaches C2.2, Q3.3 (C), R2.2, R5.1
- net BASE: now also TP5.1
- net at R26.2, R27.1: now also Q4.3 (C)
- net at C6.1, R17.2, R21.1: now also U1.5 (+)
- net at C6.2, R18.2, R22.1: now also U1.6 (-)
- net OUT_DIV: now reaches R16.1, R7.2
- net OUT_DIV: now also R11.1, TP7.1
- net at R13.1: now also U1.1
- net at R28.2: now also Q4.1 (B)
- new net: D3.1 (K), R23.2, U2.1
- new net: C1.1, R1.1, R11.2, U1.2 (-)
- new net: C7.1, R15.2, R20.1, U1.3 (+)
- new net: D1.2 (A), D2.1 (K), Q2.3 (D), R3.2, R6.2
- new net: J2.4 (SWDCLK/TCK), U3.41 (SWCLK)
- new net: J2.2 (SWDIO/TMS), U3.43 (SWDIO)
- new net +3V3: J2.1 (VTref), Q2.1 (G), R30.1, R4.1, TP11.1, U2.4, U3.36 (3V3)
- new net CSENSE_FILT: C8.1, R25.2, U3.34 (GPIO28_ADC2)
- new net ERR: C1.2, Q3.2 (E), R1.2, R19.1, TP3.1
- new net UART_RX_3V3: R24.1, U2.3, U3.7 (GPIO5)
- new net UART_RX_GND_ISOL: D3.2 (A), J1.6 (Pin_6), U2.2
- new net UART_RX_SIG_ISOL: J1.5 (Pin_5), R23.1
- new net UART_TX_3V3: Q2.2 (S), R4.2, U3.6 (GPIO4)
- new net UART_TX_SIG_5V: J1.4 (Pin_4), R6.1
- new net ~{RESET}: J2.10 (~{RESET}), R30.2, U3.30 (RUN)
- no-connect marks 0 -> 32
Other:
- note added: "C_diff2"
- note added: "Current Sense Signal Filter"
- note added: "Difference amplifier looks at difference between commanded output voltage and actual output voltage and drives base of CE amp BJT such that an error voltage Verr is proportional to the output voltage error. Verr is a current sense resistor for the CE BJT stage, so if Verr is >0V, the output stage is sourcing current into the load. V_err = (V_cmd - V_out) * (R_diff2 / R_diff1)"
- note added: "Error Amplifier"
- note added: "Filtered level shifter approximates a 5V DAC with PWM output from Pico."
- note added: "From current sense amplifier."
- note added: "I_f = 10mA for >100% CTR V_f = 1.2V"
- note added: "Input Protection Clamp"
- note added: "Isolated UART Input and Level-Shifted UART Output"
- note added: "Level shifted output asserts GND connection to next device in chain. Isolated input accepts GND connection from next device in chain."
- note added: "Optional voltage divider to add amplification to output voltage relative to V_cmd."
- note added: "Output Stage PNP CE Amp"
- note added: "Pi Pico 32-bit Microcontroller Module"
- note added: "Protection Diode"
- note added: "Pseudo DAC"
- note added: "R_diff1"
- note added: "R_diff2"
- note added: "TODO: - Protections for 5V / GND (reverse polarity etc). - Protections for OUT."
- note added: "f_c = 159Hz"
- note added: "f_c = 796Hz"
- note removed: "Compensation Network"
- note removed: "Control Op Amp"
- note removed: "Forces open loop gain to roll off before things get unstable. Prioritize low frequency open loop gain for DC stability; low bandwidth acceptable for this application."
- note removed: "LM358 is not rail to rail but should be OK since output stage is doing the actual leg work."
- note removed: "f_c = 1.59Hz"
- note removed: "f_c = 1.59kHz"
- company: (none) -> Pants for Birds
- title: (none) -> Single Cell Battery Simulator Pico Demo Board
- moved on the sheet: C2, C3, C4, C5, C6, C9, Q1, Q3, R10, R12, R13, R14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
