File: kicad/scbs_stm32g4/scbs_stm32g4.kicad_sch (KiCad schematic)
At the start: 64 parts, among them J1 Conn_01x06_Male, J2 Conn_ARM_JTAG_SWD_10, Q1 2N2907, Q2 2N7002, Q3 MMBT3904, Q4 MMBT3904, U1 TLV9062xD, U2 PC817, U3 Pico

Commit message: Add calibrated output voltage setting
* Python script serial utility for sending DIS, MWR, MRD commands to
  device.
* Three-coefficient polynomial calibration implemented in firmware for
  closer matching of output voltage (looks pretty darn good)! Makes up
  for the crappiness / non-linearity of the PWM pseudo-DAC driving a
  load without a buffer.
* Connecting the plumbing for setting output voltage via serial in the
  SCBS firmware.
* Clean up some commented code garbage that was lying around.
Parts:
- removed U3: Pico, Custom_Module:RPi_Pico_SMD_TH, symbol Custom_MCU:Pico
- added C10, C11: 6.8pF, symbol Device:C
- added C12, C13: 10uF, symbol Device:C
- added C14, C16, C17, C18, C19: 0.1uF, symbol Device:C
- added C15, C20: 1uF, symbol Device:C
- added FB1: 600R@100MHz, symbol Device:FerriteBead_Small
- added R29: 10k, symbol Device:R_US
- added U3: STM32G431CBT6, LQFP48-7x7mm, symbol stm32g4:STM32G431CBT6
- added U4: AZ1117C-3.3, symbol Regulator_Linear:AZ1117-3.3
- added Y1: 24MHz, symbol Device:Crystal
- C1, C7: value 1nF -> 0.1uF
- R1, R20: value 2M -> 2k
- R11, R15: value 10M -> 10k
Connections:
- net +3V3: now also C13.1, C16.1, C17.1, C18.1, C19.1, C20.1, FB1.1, U3.20 (VREF+), U3.24 (VDD), U3.36 (VDD), U3.48 (VDD), U4.2 (VO)
- net +5V: now also C12.1, U4.3 (VI)
- net CMD_PWM: now also U3.30 (PA8)
- net CSENSE_FILT: now also U3.10 (PA2)
- net GND: now also C10.1, C11.1, C12.2, C13.2, C14.2, C15.2, C16.2, C17.2, C18.2, C19.2, C20.2, R29.2, U3.19 (VSSA), U3.23 (VSS), U3.35 (VSS), U3.47 (VSS), U4.1 (GND)
- net UART_RX_3V3: now also U3.44 (PB7)
- net UART_TX_3V3: now also U3.43 (PB6)
- net ~{RESET}: now also U3.7 (PG10-NRST)
- net SWCLK: now reaches J2.4 (SWDCLK/TCK)
- net SWCLK: now also U3.38 (PA14)
- net SWDIO: now reaches J2.2 (SWDIO/TMS)
- net SWDIO: now also U3.37 (PA13)
- new net: C14.1, C15.1, FB1.2, U3.21 (VDDA)
- new net: C11.2, U3.6 (PF1-OSC_OUT), Y1.1
- new net: C10.2, U3.5 (PF0-OSC_IN), Y1.2
- new net: R29.1, U3.45 (PB8-BOOT0)
Other:
- note added: "f_c = 796Hz"
- note removed: "Pi Pico 32-bit Microcontroller Module"
- note removed: "f_c = 79.6Hz"
- moved on the sheet: J2, R30, TP10, TP11, TP9
