File: kicad/scbs_array/scbs_array.kicad_pcb (KiCad board)
At the start: 2 copper layers, 90 x 74 mm, 33 parts, among them J1 Barrel_Jack, J2 Phoenix MSTBA 1x05 5.08mm, J3 Conn_01x03_Male, Q1 FQP27P06, U1 WRB1205S-3WR2, U2 WRB1205S-3WR2, U3 WRB1205S-3WR2, U4 WRB1205S-3WR2

Commit message: Make enclosure CAD
Parts:
- JP1: value Jumper_2_Bridged -> 0R
- R1: value 200R -> 2k
Changed lines of the file:
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@@
       (effects (font (size 1 1) (thickness 0.15)) (justify mirror))
     )
-    (fp_text value "200R" (at 0 -1.65) (layer "B.Fab")
+    (fp_text value "2k" (at 0 -1.65) (layer "B.Fab")
       (effects (font (size 1 1) (thickness 0.15)) (justify mirror))
     )
@@
       (effects (font (size 1 1) (thickness 0.15)) (justify mirror))
     )
-    (fp_text value "Jumper_2_Bridged" (at 0 -1.65 90) (layer "B.Fab")
+    (fp_text value "0R" (at 0 -1.65 90) (layer "B.Fab")
       (effects (font (size 1 1) (thickness 0.15)) (justify mirror))
     )
